File: ArpeggiatorV1.1.kicad_sch (KiCad schematic)
At the start: 67 parts, among them J1 DIN-5_MIDI_IN, J2 DIN-5_SYNC_IN, J3 DIN-5_MIDI_OUT, J4 Conn_01x03_Pin, SW1 SW_SYNC, SW2 SW_MODE, SW3 SW_OCT, SW4 SW_ONOFF, SW5 SW_HOLD, U1 6N138, U2 6N138, U3 Pico

Commit message: Mostly finished PCB layout.
Other:
- note added: "Board-level decoupling"
- moved on the sheet: H1, H2, H3, H4, H5, H6
Changed lines of the file:
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@@
     (stroke (width 0) (type default))
   )
-  (wire (pts (xy 294.64 44.45) (xy 294.64 48.26))
+  (wire (pts (xy 294.64 44.45) (xy 294.64 45.72))
     (stroke (width 0) (type default))
   )
@@
     (effects (font (size 3 3)) (justify right bottom))
   )
+  (text "Board-level\ndecoupling" (at 298.45 49.53 0)
+    (effects (font (size 1.27 1.27)) (justify left bottom))
+  )
   (text "Buttons and LEDs" (at 194.31 238.76 0)
     (effects (font (size 3 3) (thickness 0.6) bold) (justify right bottom))
@@
     (effects (font (size 3 3)) (justify left bottom))
   )
-  (text "Debug port" (at 289.56 129.54 0)
+  (text "Debug port" (at 283.21 128.27 0)
     (effects (font (size 1.27 1.27)) (justify right bottom))
   )
@@
     )
   )
-  (symbol (lib_id "Mechanical:MountingHole") (at 342.9 58.42 0) (unit 1)
-    (in_bom yes) (on_board yes) (dnp no) (fields_autoplaced)
-    (property "Reference" "H6" (at 345.44 57.785 0)
+  (symbol (lib_id "Mechanical:MountingHole") (at 321.31 66.04 0) (unit 1)
+    (in_bom yes) (on_board yes) (dnp no) (fields_autoplaced)
+    (property "Reference" "H6" (at 323.85 65.405 0)
       (effects (font (size 1.27 1.27)) (justify left))
     )
-    (property "Value" "MountingHole" (at 345.44 60.325 0)
+    (property "Value" "MountingHole" (at 323.85 67.945 0)
       (effects (font (size 1.27 1.27)) (justify left))
     )
-    (property "Footprint" "MountingHole:MountingHole_4mm" (at 342.9 58.42 0)
-      (effects (font (size 1.27 1.27)) hide)
-    )
-    (property "Datasheet" "~" (at 342.9 58.42 0)
+    (property "Footprint" "MountingHole:MountingHole_4mm" (at 321.31 66.04 0)
+      (effects (font (size 1.27 1.27)) hide)
+    )
+    (property "Datasheet" "~" (at 321.31 66.04 0)
       (effects (font (size 1.27 1.27)) hide)
     )
@@
     )
   )
-  (symbol (lib_id "Mechanical:MountingHole") (at 342.9 39.37 0) (unit 1)
-    (in_bom yes) (on_board yes) (dnp no) (fields_autoplaced)
-    (property "Reference" "H3" (at 345.44 38.735 0)
+  (symbol (lib_id "Mechanical:MountingHole") (at 321.31 46.99 0) (unit 1)
+    (in_bom yes) (on_board yes) (dnp no) (fields_autoplaced)
+    (property "Reference" "H3" (at 323.85 46.355 0)
       (effects (font (size 1.27 1.27)) (justify left))
     )
-    (property "Value" "MountingHole" (at 345.44 41.275 0)
+    (property "Value" "MountingHole" (at 323.85 48.895 0)
       (effects (font (size 1.27 1.27)) (justify left))
     )
-    (property "Footprint" "MountingHole:MountingHole_4mm" (at 342.9 39.37 0)
-      (effects (font (size 1.27 1.27)) hide)
-    )
-    (property "Datasheet" "~" (at 342.9 39.37 0)
+    (property "Footprint" "MountingHole:MountingHole_4mm" (at 321.31 46.99 0)
+      (effects (font (size 1.27 1.27)) hide)
+    )
+    (property "Datasheet" "~" (at 321.31 46.99 0)
       (effects (font (size 1.27 1.27)) hide)
     )
@@
     )
   )
-  (symbol (lib_id "Mechanical:MountingHole") (at 342.9 45.72 0) (unit 1)
-    (in_bom yes) (on_board yes) (dnp no) (fields_autoplaced)
-    (property "Reference" "H4" (at 345.44 45.085 0)
+  (symbol (lib_id "Mechanical:MountingHole") (at 321.31 53.34 0) (unit 1)
+    (in_bom yes) (on_board yes) (dnp no) (fields_autoplaced)
+    (property "Reference" "H4" (at 323.85 52.705 0)
       (effects (font (size 1.27 1.27)) (justify left))
     )
-    (property "Value" "MountingHole" (at 345.44 47.625 0)
+    (property "Value" "MountingHole" (at 323.85 55.245 0)
       (effects (font (size 1.27 1.27)) (justify left))
     )
-    (property "Footprint" "MountingHole:MountingHole_4mm" (at 342.9 45.72 0)
-      (effects (font (size 1.27 1.27)) hide)
-    )
-    (property "Datasheet" "~" (at 342.9 45.72 0)
+    (property "Footprint" "MountingHole:MountingHole_4mm" (at 321.31 53.34 0)
+      (effects (font (size 1.27 1.27)) hide)
+    )
+    (property "Datasheet" "~" (at 321.31 53.34 0)
       (effects (font (size 1.27 1.27)) hide)
     )
@@
     )
   )
-  (symbol (lib_id "Mechanical:MountingHole") (at 342.9 33.02 0) (unit 1)
-    (in_bom yes) (on_board yes) (dnp no) (fields_autoplaced)
-    (property "Reference" "H2" (at 345.44 32.385 0)
+  (symbol (lib_id "Mechanical:MountingHole") (at 321.31 40.64 0) (unit 1)
+    (in_bom yes) (on_board yes) (dnp no) (fields_autoplaced)
+    (property "Reference" "H2" (at 323.85 40.005 0)
       (effects (font (size 1.27 1.27)) (justify left))
     )
-    (property "Value" "MountingHole" (at 345.44 34.925 0)
+    (property "Value" "MountingHole" (at 323.85 42.545 0)
       (effects (font (size 1.27 1.27)) (justify left))
     )
-    (property "Footprint" "MountingHole:MountingHole_4mm" (at 342.9 33.02 0)
-      (effects (font (size 1.27 1.27)) hide)
-    )
-    (property "Datasheet" "~" (at 342.9 33.02 0)
+    (property "Footprint" "MountingHole:MountingHole_4mm" (at 321.31 40.64 0)
+      (effects (font (size 1.27 1.27)) hide)
+    )
+    (property "Datasheet" "~" (at 321.31 40.64 0)
       (effects (font (size 1.27 1.27)) hide)
     )
@@
     )
   )
-  (symbol (lib_id "Mechanical:MountingHole") (at 342.9 52.07 0) (unit 1)
-    (in_bom yes) (on_board yes) (dnp no) (fields_autoplaced)
-    (property "Reference" "H5" (at 345.44 51.435 0)
+  (symbol (lib_id "Mechanical:MountingHole") (at 321.31 59.69 0) (unit 1)
+    (in_bom yes) (on_board yes) (dnp no) (fields_autoplaced)
+    (property "Reference" "H5" (at 323.85 59.055 0)
       (effects (font (size 1.27 1.27)) (justify left))
     )
-    (property "Value" "MountingHole" (at 345.44 53.975 0)
+    (property "Value" "MountingHole" (at 323.85 61.595 0)
       (effects (font (size 1.27 1.27)) (justify left))
     )
-    (property "Footprint" "MountingHole:MountingHole_4mm" (at 342.9 52.07 0)
-      (effects (font (size 1.27 1.27)) hide)
-    )
-    (property "Datasheet" "~" (at 342.9 52.07 0)
+    (property "Footprint" "MountingHole:MountingHole_4mm" (at 321.31 59.69 0)
+      (effects (font (size 1.27 1.27)) hide)
+    )
+    (property "Datasheet" "~" (at 321.31 59.69 0)
       (effects (font (size 1.27 1.27)) hide)
     )
@@
     )
   )
-  (symbol (lib_id "Mechanical:MountingHole") (at 342.9 26.67 0) (unit 1)
-    (in_bom yes) (on_board yes) (dnp no) (fields_autoplaced)
-    (property "Reference" "H1" (at 345.44 26.035 0)
+  (symbol (lib_id "Mechanical:MountingHole") (at 321.31 34.29 0) (unit 1)
+    (in_bom yes) (on_board yes) (dnp no) (fields_autoplaced)
+    (property "Reference" "H1" (at 323.85 33.655 0)
       (effects (font (size 1.27 1.27)) (justify left))
     )
-    (property "Value" "MountingHole" (at 345.44 28.575 0)
+    (property "Value" "MountingHole" (at 323.85 36.195 0)
       (effects (font (size 1.27 1.27)) (justify left))
     )
-    (property "Footprint" "MountingHole:MountingHole_4mm" (at 342.9 26.67 0)
-      (effects (font (size 1.27 1.27)) hide)
-    )
-    (property "Datasheet" "~" (at 342.9 26.67 0)
+    (property "Footprint" "MountingHole:MountingHole_4mm" (at 321.31 34.29 0)
+      (effects (font (size 1.27 1.27)) hide)
+    )
+    (property "Datasheet" "~" (at 321.31 34.29 0)
       (effects (font (size 1.27 1.27)) hide)
     )
@@
     )
   )
-  (symbol (lib_id "power:GND") (at 294.64 48.26 0) (unit 1)
-    (in_bom yes) (on_board yes) (dnp no) (fields_autoplaced)
-    (property "Reference" "#PWR024" (at 294.64 54.61 0)
-      (effects (font (size 1.27 1.27)) hide)
-    )
-    (property "Value" "GND" (at 294.64 53.34 0)
-      (effects (font (size 1.27 1.27)))
-    )
-    (property "Footprint" "" (at 294.64 48.26 0)
-      (effects (font (size 1.27 1.27)) hide)
-    )
-    (property "Datasheet" "" (at 294.64 48.26 0)
+  (symbol (lib_id "power:GND") (at 294.64 45.72 0) (unit 1)
+    (in_bom yes) (on_board yes) (dnp no) (fields_autoplaced)
+    (property "Reference" "#PWR024" (at 294.64 52.07 0)
+      (effects (font (size 1.27 1.27)) hide)
+    )
+    (property "Value" "GND" (at 294.64 50.8 0)
+      (effects (font (size 1.27 1.27)))
+    )
+    (property "Footprint" "" (at 294.64 45.72 0)
+      (effects (font (size 1.27 1.27)) hide)
+    )
+    (property "Datasheet" "" (at 294.64 45.72 0)
       (effects (font (size 1.27 1.27)) hide)
     )
@@
   )
   (symbol (lib_id "power:GND") (at 266.7 46.99 0) (unit 1)
-    (in_bom yes) (on_board yes) (dnp no) (fields_autoplaced)
+    (in_bom yes) (on_board yes) (dnp no)
     (property "Reference" "#PWR020" (at 266.7 53.34 0)
       (effects (font (size 1.27 1.27)) hide)
     )
-    (property "Value" "GND" (at 266.7 52.07 0)
-      (effects (font (size 1.27 1.27)))
-    )
+    (property "Value" "GND" (at 269.24 46.99 0)
+      (effects (font (size 1.27 1.27)))
+    )
